File: ESP32-S2-Breakout/ESP32-S2-Breakout.kicad_pcb (KiCad board)
At the start: 2 copper layers, 55.9 x 30.5 mm, 37 parts, among them J1 USB_B_Micro, J2 Conn_01x21, J3 Conn_01x21, SW1 Reset, SW2 Boot, U1 USBLC6-2SC6, U2 ESP32-S2-WROOM, U3 XC6220B331MR, Y1 32.768KHz

Commit message: Add resistor values for 1.8V/2mA LEDs
Parts:
- R5: value TBD -> 750r
- R9: value TBD -> 1.6k
Changed lines of the file:
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@@
       (effects (font (size 0.6 0.6) (thickness 0.15)))
     )
-    (fp_text value TBD (at 0 1.43) (layer F.Fab)
+    (fp_text value 1.6k (at 0 1.43) (layer F.Fab)
       (effects (font (size 1 1) (thickness 0.15)))
     )
@@
       (effects (font (size 0.6 0.6) (thickness 0.15)))
     )
-    (fp_text value TBD (at 0 1.43) (layer F.Fab)
-      (effects (font (size 1 1) (thickness 0.15)))
-    )
+    (fp_text value 750r (at 0 1.43) (layer F.Fab)
+      (effects (font (size 1 1) (thickness 0.15)))
+    )

Commit message: Add USB series termination resistor and bypass capacitor values
Parts:
- C10, C9: value TBD -> 20p
- R6, R7: value TBD -> 22r
Changed lines of the file:
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@@
       (effects (font (size 0.6 0.6) (thickness 0.15)))
     )
-    (fp_text value TBD (at 0 1.43 90) (layer F.Fab)
+    (fp_text value 20p (at 0 1.43 90) (layer F.Fab)
       (effects (font (size 1 1) (thickness 0.15)))
     )
@@
       (effects (font (size 0.6 0.6) (thickness 0.15)))
     )
-    (fp_text value TBD (at 0 1.43 90) (layer F.Fab)
+    (fp_text value 20p (at 0 1.43 90) (layer F.Fab)
       (effects (font (size 1 1) (thickness 0.15)))
     )
@@
       (effects (font (size 0.6 0.6) (thickness 0.15)))
     )
-    (fp_text value TBD (at 0 1.43) (layer F.Fab)
+    (fp_text value 22r (at 0 1.43) (layer F.Fab)
       (effects (font (size 1 1) (thickness 0.15)))
     )
@@
       (effects (font (size 0.6 0.6) (thickness 0.15)))
     )
-    (fp_text value TBD (at 0 1.43) (layer F.Fab)
-      (effects (font (size 1 1) (thickness 0.15)))
-    )
+    (fp_text value 22r (at 0 1.43) (layer F.Fab)
+      (effects (font (size 1 1) (thickness 0.15)))
+    )

Commit message: Add resistor and capacitor values for 32.758kHz crystal
Parts:
- CL1, CL2: value TBD -> 11p C0G
- R1: value TBD -> N/C
- R2, R3: value TBD -> 220r 1%
Changed lines of the file:
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@@
       (effects (font (size 0.6 0.6) (thickness 0.15)))
     )
-    (fp_text value TBD (at 0 1.43) (layer F.Fab)
+    (fp_text value "220r 1%" (at 0 1.43) (layer F.Fab)
       (effects (font (size 1 1) (thickness 0.15)))
     )
@@
       (effects (font (size 0.6 0.6) (thickness 0.15)))
     )
-    (fp_text value TBD (at 0 1.43) (layer F.Fab)
+    (fp_text value "220r 1%" (at 0 1.43) (layer F.Fab)
       (effects (font (size 1 1) (thickness 0.15)))
     )
@@
       (effects (font (size 0.6 0.6) (thickness 0.15)))
     )
-    (fp_text value TBD (at 0 1.43 90) (layer F.Fab)
+    (fp_text value N/C (at 0 1.43 90) (layer F.Fab)
       (effects (font (size 1 1) (thickness 0.15)))
     )
@@
       (effects (font (size 0.6 0.6) (thickness 0.15)))
     )
-    (fp_text value TBD (at 0 1.43) (layer F.Fab)
+    (fp_text value "11p C0G" (at 0 1.43) (layer F.Fab)
       (effects (font (size 1 1) (thickness 0.15)))
     )
@@
       (effects (font (size 0.6 0.6) (thickness 0.15)))
     )
-    (fp_text value TBD (at 0 1.43) (layer F.Fab)
-      (effects (font (size 1 1) (thickness 0.15)))
-    )
+    (fp_text value "11p C0G" (at 0 1.43) (layer F.Fab)
+      (effects (font (size 1 1) (thickness 0.15)))
+    )

Commit message: Add values for ferrite bead on usb connector
Parts:
- C1: value TBD -> 0.1u
- FB1, FB2: value TBD -> >1A
Changed lines of the file:
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@@
       (effects (font (size 0.6 0.6) (thickness 0.15)))
     )
-    (fp_text value TBD (at 0 1.43) (layer F.Fab)
+    (fp_text value >1A (at 0 1.43) (layer F.Fab)
       (effects (font (size 1 1) (thickness 0.15)))
     )
@@
       (effects (font (size 0.6 0.6) (thickness 0.15)))
     )
-    (fp_text value TBD (at 0 1.43) (layer F.Fab)
+    (fp_text value 0.1u (at 0 1.43) (layer F.Fab)
       (effects (font (size 1 1) (thickness 0.15)))
     )
@@
       (effects (font (size 0.6 0.6) (thickness 0.15)))
     )
-    (fp_text value TBD (at 0 1.43) (layer F.Fab)
-      (effects (font (size 1 1) (thickness 0.15)))
-    )
+    (fp_text value >1A (at 0 1.43) (layer F.Fab)
+      (effects (font (size 1 1) (thickness 0.15)))
+    )
