File: ESP32-S2-Breakout/ESP32-S2-Breakout.sch (KiCad schematic (older format))
At the start: 36 parts, among them J1 USB_B_Micro, J3 Conn_01x23, SW1 Reset, SW2 Boot, U1 USBLC6-2SC6, U2 ESP32-S2-WROOM, U3 XC6220B331MR, Y1 32.768KHz

Commit message: Rev 2/v2 update
Parts:
- removed J1: USB_B_Micro, Connector_USB:USB_Micro-B_Molex-105017-0001, symbol Connector:USB_B_Micro
- added J1: USB_C_Receptacle_USB2.0, ESP32-S2-Breakout:USB_C_Receptacle_HRO_TYPE-C-31-M-12, symbol Connector:USB_C_Receptacle_USB2.0
- added R10, R11: 5.1k, Resistor_SMD:R_0603_1608Metric, symbol Device:R_Small
- C1, C11, C3, C4, C5, C6: footprint Capacitor_SMD:C_0805_2012Metric -> Capacitor_SMD:C_0603_1608Metric; LCSC (none) -> C14663
- C10, C9: footprint Capacitor_SMD:C_0805_2012Metric -> Capacitor_SMD:C_0603_1608Metric; LCSC (none) -> C1648
- C2: footprint Capacitor_SMD:C_0805_2012Metric -> Capacitor_SMD:C_0603_1608Metric; LCSC (none) -> C84419
- C7: footprint Capacitor_SMD:C_0805_2012Metric -> Capacitor_SMD:C_0603_1608Metric; LCSC (none) -> C90058
- C8: footprint Capacitor_SMD:C_0805_2012Metric -> Capacitor_SMD:C_0603_1608Metric; LCSC (none) -> C69335
- CL1, CL2: value TBD -> 20p; footprint Capacitor_SMD:C_0805_2012Metric -> Capacitor_SMD:C_0603_1608Metric; LCSC (none) -> C1648
- D1: footprint LED_SMD:LED_0805_2012Metric -> LED_SMD:LED_0603_1608Metric; LCSC (none) -> C205443
- D2: footprint LED_SMD:LED_0805_2012Metric -> LED_SMD:LED_0603_1608Metric; LCSC (none) -> C205445
- FB1, FB2: footprint Inductor_SMD:L_0805_2012Metric -> Inductor_SMD:L_0603_1608Metric; LCSC (none) -> C24821
- R1: value TBD -> N/C; footprint Resistor_SMD:R_0805_2012Metric -> Resistor_SMD:R_0603_1608Metric; LCSC (none) -> -
- R2, R3: value TBD -> 0r; footprint Resistor_SMD:R_0805_2012Metric -> Resistor_SMD:R_0603_1608Metric; LCSC (none) -> C21189
- R4, R8: footprint Resistor_SMD:R_0805_2012Metric -> Resistor_SMD:R_0603_1608Metric; LCSC (none) -> C99198
- R5: value 750r -> 100r; footprint Resistor_SMD:R_0805_2012Metric -> Resistor_SMD:R_0603_1608Metric; LCSC (none) -> C22775
- R6, R7: footprint Resistor_SMD:R_0805_2012Metric -> Resistor_SMD:R_0603_1608Metric; LCSC (none) -> C23345
- R9: value 1.6k -> 100r; footprint Resistor_SMD:R_0805_2012Metric -> Resistor_SMD:R_0603_1608Metric; LCSC (none) -> C22775
- SW1, SW2: footprint Button_Switch_SMD:SW_Push_SPST_NO_Alps_SKRK -> ESP32-S2-Breakout:Alps_SKRK; LCSC (none) -> C115357
- U1: LCSC (none) -> C7519
- U2: footprint ESP32-S2-WROOM:ESP32-S2-WROOM -> ESP32-S2-Breakout:ESP32-S2-WROOM; LCSC (none) -> C701327
- U3: symbol Regulator_Linear:XC6220B331MR -> ESP32-S2-Breakout-rescue:XC6220B331MR-Regulator_Linear; LCSC (none) -> C86534
- Y1: value 32.768KHz -> 32.768KHz 12.5p; footprint Crystal:Crystal_SMD_3215-2Pin_3.2x1.5mm -> ESP32-S2-Breakout:Crystal_SMD_3215-2Pin_3.2x1.5mm; LCSC (none) -> C271654
- renumbered e1 to J2
Connections:
- net +3V3: now also JP1.1 (A)
- net +5V: no longer JP1.1 (A)
- net D+: now also J1.A6 (D+), J1.B6 (D+)
- net D-: now also J1.A7 (D-), J1.B7 (D-)
- net GND: now also C1.1, FB1.2, J1.A1 (GND), J1.A12 (GND), J1.B1 (GND), J1.B12 (GND), R10.2, R11.2; no longer C1.2, FB1.1
- net VBUS: now also J1.A4 (VBUS), J1.A9 (VBUS), J1.B4 (VBUS), J1.B9 (VBUS)
- new net: C1.2, FB1.1, J1.S1 (SHIELD)
- new net: J1.A5 (CC1), R11.1
- new net: J1.B5 (CC2), R10.1
- no-connect marks 1 -> 2
Other:
- note removed: "Assume LED\n 1.8V 2mA"
- moved on the sheet: C1, C10, C11, C2, C3, C4, C5, C6, C9, CL1, CL2, D1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
